Commit message: atlas_v5: fix mirrored left-arm visual meshes and add compensating joint-frame rotation
Every left-arm link (clav, scap, uarm, larm, ufarm, lfarm) had its
<visual><mesh> pointing at the right arms mesh file instead of the
correctly-named l_*.dae sitting right next to it - traced via git log -p
to eb29fe8a ("apply patch from tkoolen that works better than mine"),
which flipped these while otherwise fixing real inertia/collision bugs.

Fixing the filename alone was not enough: l_arm_shz carries an extra
rpy="0 0 pi" versus r_arm_shzs identity, and l_arm_wry/l_arm_wry2
carry an extra rpy="0 pi 0" versus their right-arm counterparts
identity - the left and right arm chains use different joint-frame
conventions, not a simple bilateral mirror. Added a compensating visual
origin rotation per link: rpy="0 0 pi" for clav/scap/uarm/larm (cancels
the shz flip alone), rpy="pi 0 0" for ufarm/lfarm (shz and wry flips
compose to a net 180 flip about X).

Verified by spawning atlas_v5 directly via xacro (bypassing the
create_atlas_urdf.py-generated URDF) in gz sim and visually confirming
the left arm now mirrors the right.

File: atlas_description/urdf/atlas_v5_simple_shapes.urdf (robot description, URDF)
Before this commit: robot drc_skeleton, 34 links, 34 joints
Links:
- link l_clav: geometry collision box size=0.1 0.07 0.072; collision cylinder length=0.1525 radius=0.0555
- link l_larm: geometry collision box size=0.025 0.06 0.06; collision box size=0.025 0.155 0.07
- link l_lfarm: geometry collision cylinder length=0.015 radius=0.045; collision cylinder length=0.015 radius=0.052
- link l_scap: geometry collision box size=0.02 0.029 0.018; collision box size=0.028 0.090 0.05
- link l_uarm: geometry collision box size=0.05 0.07 0.15; collision cylinder length=0.11 radius=0.065
- link l_ufarm: geometry collision box size=0.08 0.09 0.11; collision cylinder length=0.1 radius=0.053
