Commit message: atlas_v4: fix mirrored left-arm visual meshes and add compensating joint-frame rotation
Same bug and fix as cf780453 (atlas_v5): every left-arm link (clav,
scap, uarm, larm, ufarm, lfarm) had its <visual><mesh> pointing at the
right arms mesh file instead of the correctly-named l_*.dae, and
l_arm_shz/l_arm_wry/l_arm_wry2 carry the same extra rpy="0 0 pi" /
rpy="0 pi 0" versus their right-arm counterparts identity that v5 has.
Applied the same compensating visual origin rotation: rpy="0 0 pi" for
clav/scap/uarm/larm, rpy="pi 0 0" for ufarm/lfarm.

Verified by spawning atlas_v4 directly via xacro in gz sim and visually
confirming the left arm now mirrors the right.

File: atlas_description/urdf/atlas_v4_simple_shapes.urdf (robot description, URDF)
Before this commit: robot drc_skeleton, 34 links, 34 joints
Links:
- link l_clav: geometry collision box size=0.1 0.07 0.072; collision cylinder length=0.1525 radius=0.0555
- link l_larm: geometry collision box size=0.135 0.15 0.06; collision cylinder length=0.125 radius=0.045
- link l_lfarm: geometry collision box size=0.13 0.09 0.07; collision cylinder length=0.05 radius=0.03
- link l_scap: geometry collision box size=0.02 0.029 0.018; collision box size=0.028 0.090 0.05
- link l_uarm: geometry collision box size=0.05 0.07 0.15; collision cylinder length=0.11 radius=0.065
- link l_ufarm: geometry collision box size=0.135 0.1 0.045; collision cylinder length=0.125 radius=0.045
