Commit message: remove empty collision box

File: irobot_hand_description/urdf/irobot_hand.urdf.xacro (robot description, xacro)
@@ -64,10 +64,4 @@
                izz="${2.65921e-7 / (2 * flex_joint_steps + 1)}"/>
     </inertial>
-    <collision>
-      <geometry>
-        <box size="0 0 0"/>
-      </geometry>
-      <origin xyz="0 0 0" rpy="0 0 0"/>
-    </collision>
     <visual>
       <geometry>
@@ -114,10 +108,4 @@
                izz="${2.65921e-7 / (2 * flex_joint_steps + 1)}"/>
     </inertial>
-    <collision>
-      <geometry>
-        <box size="0 0 0"/>
-      </geometry>
-      <origin xyz="0 0 0" rpy="0 0 0"/>
-    </collision>
     <visual>
       <geometry>
@@ -161,10 +149,4 @@
                izz="${2.65921e-7 / (2 * flex_joint_steps + 1)}"/>
     </inertial>
-    <collision>
-      <geometry>
-        <box size="0 0 0"/>
-      </geometry>
-      <origin xyz="0 0 0" rpy="0 0 0"/>
-    </collision>
     <visual>
       <geometry>

Commit message: changed inertial to equivalent solid-box inertia

File: irobot_hand_description/urdf/irobot_hand.urdf.xacro (robot description, xacro)
@@ -360,11 +360,6 @@
       <inertial>
         <mass value="0.0288"/>
-        <!-- gazebo -> cad coordinate mapping
-             x -> -y
-             y -> -z
-             z -> x
-        -->
-        <origin xyz="-0.002630 0.002396 0.021770" rpy="${pi/2} -${pi/2} 0"/>
-        <inertia ixx="2.420689e-6" ixy="-1.449042e-6" ixz="-7.74579e-7" iyy="1.196202e-6" iyz="1.90704e-7" izz="1.2736461e-6"/>
+        <origin xyz="0 0.0028 0.033" rpy="0 0 0"/>
+        <inertia ixx="8.126e-6" ixy="0" ixz="0" iyy="8.038e-6" iyz="0" izz="1.644e-6"/>
       </inertial>
     <xacro:proximal_link_collisions/>
@@ -433,11 +428,6 @@
       <inertial>
         <mass value="0.0288"/>
-        <!-- gazebo -> cad coordinate mapping
-             x -> -y
-             y -> -z
-             z -> x
-        -->
-        <origin xyz="-0.002630 0.002396 0.021770" rpy="${pi/2} -${pi/2} 0"/>
-        <inertia ixx="2.420689e-6" ixy="-1.449042e-6" ixz="-7.74579e-7" iyy="1.196202e-6" iyz="1.90704e-7" izz="1.2736461e-6"/>
+        <origin xyz="0 0.0028 0.033" rpy="0 0 0"/>
+        <inertia ixx="8.126e-6" ixy="0" ixz="0" iyy="8.038e-6" iyz="0" izz="1.644e-6"/>
       </inertial>
     <xacro:proximal_link_collisions/>
@@ -489,11 +479,6 @@
       <inertial>
         <mass value="0.0288"/>
-        <!-- gazebo -> cad coordinate mapping
-             x -> -y
-             y -> -z
-             z -> x
-        -->
-        <origin xyz="-0.002630 0.002396 0.021770" rpy="${pi/2} -${pi/2} 0"/>
-        <inertia ixx="2.420689e-6" ixy="-1.449042e-6" ixz="-7.74579e-7" iyy="1.196202e-6" iyz="1.90704e-7" izz="1.2736461e-6"/>
+        <origin xyz="0 0.0028 0.033" rpy="0 0 0"/>
+        <inertia ixx="8.126e-6" ixy="0" ixz="0" iyy="8.038e-6" iyz="0" izz="1.644e-6"/>
       </inertial>
     <xacro:proximal_link_collisions/>

Commit message: don't redefine pi

File: irobot_hand_description/urdf/irobot_hand.urdf.xacro (robot description, xacro)
@@ -7,5 +7,4 @@
 <xacro:property name="flex_joint_steps" value="2" />
 <xacro:property name="proximal_link_length" value=".062" />
-<xacro:property name="pi" value="3.14" />
 <xacro:property name="flex_offset" value="0.003"/> <!--${0.5*flex_joint_length/flex_joint_steps}-->
 <xacro:macro name="flex_link" params="side finger_id link_id">

Commit message: remove zero-size box visuals from hidden flex-joint links

File: irobot_hand_description/urdf/irobot_hand.urdf.xacro (robot description, xacro)
@@ -63,10 +63,4 @@
                izz="${2.65921e-7 / (2 * flex_joint_steps + 1)}"/>
     </inertial>
-    <visual>
-      <geometry>
-        <box size="0 0 0"/>
-      </geometry>
-      <origin xyz="0 0 0" rpy="0 0 0"/>
-    </visual>
   </link>
   <gazebo reference="${side}_finger[${finger_id}]/flexible_joint_twist_from_${link_from}_to_${link_to}">
@@ -107,10 +101,4 @@
                izz="${2.65921e-7 / (2 * flex_joint_steps + 1)}"/>
     </inertial>
-    <visual>
-      <geometry>
-        <box size="0 0 0"/>
-      </geometry>
-      <origin xyz="0 0 0" rpy="0 0 0"/>
-    </visual>
   </link>
   <gazebo reference="${side}_finger[${finger_id}]/flexible_joint_twist_from_proximal_to_1">
@@ -148,10 +136,4 @@
                izz="${2.65921e-7 / (2 * flex_joint_steps + 1)}"/>
     </inertial>
-    <visual>
-      <geometry>
-        <box size="0 0 0"/>
-      </geometry>
-      <origin xyz="0 0 0" rpy="0 0 0"/>
-    </visual>
   </link>
   <gazebo reference="${side}_finger[${finger_id}]/flexible_joint_twist_from_${flex_joint_steps}_to_distal">

Commit message: replace legacy gearbox spread coupling with mimic joint
The Gazebo-classic gearbox extension made finger[1]/base_rotation_link
a child of finger[0]/base_rotation_link in addition to its existing
parent joint from base_link. gz-sim enforces a strict
single-parent kinematic tree. A <mimic> tag constrains
joint position rather than link parentage, avoiding the conflict.

File: irobot_hand_description/urdf/irobot_hand.urdf.xacro (robot description, xacro)
@@ -537,27 +537,6 @@
     <axis xyz="0 0 1"/>
     <limit effort="1000.0" lower="0.0" upper="${pi/2}" velocity="0.5"/>
-  </joint>
-  <gazebo>
-    <joint name="${side}_spread_gearbox" type="gearbox">
-      <parent>${side}_finger[0]/base_rotation_link</parent>
-      <child>${side}_finger[1]/base_rotation_link</child>
-      <!-- ${side}_base_link got lumped into ${parent},
-           so we need to fix parser_urdf.cc to propagate name
-           changes into this extension before switching this
-           to use ${side_base_link}. -->
-      <gearbox_reference_body>${parent}</gearbox_reference_body>
-      <gearbox_ratio>1.0</gearbox_ratio>
-      <axis>
-        <!-- yikes, what coordinate frame is this specified in?
-             0 0 1 causes NaNs. 0 1 0 works, but unsure why yet.-->
-        <xyz>0 1 0</xyz>
-      </axis>
-      <axis2>
-        <!-- yikes, what coordinate frame is this specified in?
-             0 0 1 causes NaNs. 0 1 0 works, but unsure why yet.-->
-        <xyz>0 1 0</xyz>
-      </axis2>
-    </joint>
-  </gazebo>
+    <mimic joint="${side}_finger[0]/joint_base_rotation" multiplier="1.0" offset="0.0"/>
+  </joint>
   <gazebo reference="${side}_finger[1]/joint_base">
     <implicitSpringDamper>1</implicitSpringDamper>
